File: hardware/soil-moisture-sensor.sch (KiCad schematic (older format))
At the start: 18 parts, among them J1 AVR ISP, J2 FTDI, SW1 SW_Push, U1 ATmega328P-AU, U2 NRF24L01_Breakout, U3 ATSHA204A, Y1 Resonator

Commit message: Add some missing LCSC part numbers and datasheets
Parts:
- J1, J2: LCSC (none) -> C2833331
Changed lines of the file:
@@
 F 2 "Connector_PinHeader_2.54mm:PinHeader_1x06_P2.54mm_Vertical" H 1150 4900 50  0001 C CNN
 F 3 "~" H 1150 4900 50  0001 C CNN
+F 4 "C2833331" H 1150 4900 50  0001 C CNN "LCSC"
 	1    1150 4900
 	1    0    0    -1
@@
 F 1 "Battery_Cell" V 5750 3150 50  0000 L CNN
 F 2 "MyFootprints:BatteryHolder_Keystone_597_591_2AAA_3V" V 5600 3410 50  0001 C CNN
-F 3 "~" V 5600 3410 50  0001 C CNN
+F 3 "https://www.keyelco.com/userAssets/file/M65p11.pdf" V 5600 3410 50  0001 C CNN
 	1    5600 3350
 	0    -1   -1   0
@@
 F 2 "Connector_PinHeader_2.54mm:PinHeader_1x06_P2.54mm_Vertical" H 1150 4000 50  0001 C CNN
 F 3 "~" H 1150 4000 50  0001 C CNN
+F 4 "C2833331" H 1150 4000 50  0001 C CNN "LCSC"
 	1    1150 4000
 	1    0    0    -1
