File: hardware/soil-moisture-sensor.sch (KiCad schematic (older format))
At the start: 18 parts, among them J1 AVR ISP, J2 FTDI, SW1 SW_Push, U1 ATmega328P-AU, U2 NRF24L01_Breakout, U3 ATSHA204A, Y1 Resonator

Commit message: Fix wrong LCSC part number
Parts:
- R4: LCSC C17514 -> C17414
Changed lines of the file:
@@
 F 2 "Resistor_SMD:R_0805_2012Metric_Pad1.15x1.40mm_HandSolder" V 9930 2600 50  0001 C CNN
 F 3 "~" H 10000 2600 50  0001 C CNN
-F 4 "C17514" V 10000 2600 50  0001 C CNN "LCSC"
+F 4 "C17414" V 10000 2600 50  0001 C CNN "LCSC"
 	1    10000 2600
 	-1   0    0    1

Commit message: Update footprint of NRF24L01-SMD
Parts:
- U2: footprint mysensors_radios:NRF24L01-SMD -> local_footprints:NRF24L01-SMD
Changed lines of the file:
@@
 F 0 "U2" H 2180 1796 50  0000 L CNN
 F 1 "NRF24L01_Breakout" H 2180 1705 50  0000 L CNN
-F 2 "mysensors_radios:NRF24L01-SMD" H 1950 2350 50  0001 L CIN
+F 2 "local_footprints:NRF24L01-SMD" H 1950 2350 50  0001 L CIN
 F 3 "http://www.nordicsemi.com/eng/content/download/2730/34105/file/nRF24L01_Product_Specification_v2_0.pdf" H 1800 1650 50  0001 C CNN
 	1    1800 1750

Commit message: Add config with "rotated" tag
The +rotated tag will be used for selecting the right components when
generating the JLCPCB pick and place files.
Parts:
- C1, C2, C3, C4, D1, J1, J2, R1, R2, R3, R4, SW1, U1, U3, Y1: Config (none) -> +rotated
Changed lines of the file:
@@
 F 3 "~" H 5550 4550 50  0001 C CNN
 F 4 "C720477" H 5550 4350 50  0001 C CNN "LCSC"
+F 5 "+rotated" H 5550 4350 50  0001 C CNN "Config"
 	1    5550 4350
 	-1   0    0    1
@@
 F 3 "~" H 1150 4900 50  0001 C CNN
 F 4 "C2833331" H 1150 4900 50  0001 C CNN "LCSC"
+F 5 "+rotated" H 1150 4900 50  0001 C CNN "Config"
 	1    1150 4900
 	1    0    0    -1
@@
 F 3 "~" H 1650 6700 50  0001 C CNN
 F 4 "C17414" V 1650 6700 50  0001 C CNN "LCSC"
+F 5 "+rotated" H 1650 6700 50  0001 C CNN "Config"
 	1    1650 6700
 	0    1    1    0
@@
 F 3 "~" H 2500 6700 50  0001 C CNN
 F 4 "C154819" H 2500 6700 50  0001 C CNN "LCSC"
+F 5 "+rotated" H 2500 6700 50  0001 C CNN "Config"
 	1    2500 6700
 	-1   0    0    1
@@
 F 3 "~" H 2850 7050 50  0001 C CNN
 F 4 "C28323" H 2850 7050 50  0001 C CNN "LCSC"
+F 5 "+rotated" H 2850 7050 50  0001 C CNN "Config"
 	1    2850 7050
 	1    0    0    -1
@@
 F 3 "~" H 3250 7050 50  0001 C CNN
 F 4 "C17733" H 3250 7050 50  0001 C CNN "LCSC"
+F 5 "+rotated" H 3250 7050 50  0001 C CNN "Config"
 	1    3250 7050
 	-1   0    0    1
@@
 F 3 "~" H 2800 1800 50  0001 C CNN
 F 4 "C127327" H 2800 1800 50  0001 C CNN "LCSC"
+F 5 "+rotated" H 2800 1800 50  0001 C CNN "Config"
 	1    2800 1800
 	-1   0    0    1
@@
 F 3 "~" H 3300 1800 50  0001 C CNN
 F 4 "C28323" H 3300 1800 50  0001 C CNN "LCSC"
+F 5 "+rotated" H 3300 1800 50  0001 C CNN "Config"
 	1    3300 1800
 	1    0    0    -1
@@
 F 3 "~" H 5500 3900 50  0001 C CNN
 F 4 "C17414" V 5500 3900 50  0001 C CNN "LCSC"
+F 5 "+rotated" H 5500 3900 50  0001 C CNN "Config"
 	1    5500 3900
 	0    1    1    0
@@
 F 3 "~" H 1150 4000 50  0001 C CNN
 F 4 "C2833331" H 1150 4000 50  0001 C CNN "LCSC"
+F 5 "+rotated" H 1150 4000 50  0001 C CNN "Config"
 	1    1150 4000
 	1    0    0    -1
@@
 F 3 "http://ww1.microchip.com/downloads/en/DeviceDoc/ATmega328_P%20AVR%20MCU%20with%20picoPower%20Technology%20Data%20Sheet%2040001984A.pdf" H 8400 2900 50  0001 C CNN
 F 4 "C14877" H 8400 2900 50  0001 C CNN "LCSC"
+F 5 "+rotated" H 8400 2900 50  0001 C CNN "Config"
 	1    8400 2900
 	1    0    0    -1
@@
 F 3 "http://www.atmel.com/Images/Atmel-8885-CryptoAuth-ATSHA204A-Datasheet.pdf" H 10680 2824 60  0001 L CNN
 F 4 "C34377" H 10650 2900 50  0001 C CNN "LCSC"
+F 5 "+rotated" H 10650 2900 50  0001 C CNN "Config"
 	1    10650 2900
 	1    0    0    -1
@@
 F 3 "~" H 10000 2600 50  0001 C CNN
 F 4 "C17414" V 10000 2600 50  0001 C CNN "LCSC"
+F 5 "+rotated" H 10000 2600 50  0001 C CNN "Config"
 	1    10000 2600
 	-1   0    0    1
@@
 F 3 "~" H 9625 2050 50  0001 C CNN
 F 4 "C907975" H 9650 2050 50  0001 C CNN "LCSC"
+F 5 "+rotated" H 9650 2050 50  0001 C CNN "Config"
 	1    9650 2050
 	-1   0    0    1
@@
 F 3 "~" H 1750 4300 50  0001 C CNN
 F 4 "C49678" V 1750 4300 50  0001 C CNN "LCSC"
+F 5 "+rotated" H 1750 4300 50  0001 C CNN "Config"
 	1    1750 4300
 	0    1    1    0
